Commit message: aruco models

File: src/agv_ugv/ugv/src/urdf/leo.urdf (robot description, URDF)
Before this commit: robot leo, 12 links, 11 joints
Links:
- link chassis: geometry collision mesh filename=package://ugv/src/meshes/Chassis_outline.stl; visual mesh filename=package://ugv/src/meshes/Chassis.dae
- link landing_pad: mass 0.001 -> 0.01; geometry collision box size=0.3 0.3 0.01; visual box size=0.3 0.3 0.01

Commit message: edit ugv

File: src/agv_ugv/ugv/src/urdf/leo.urdf (robot description, URDF)
Before this commit: robot leo, 12 links, 11 joints
Links:
- link chassis: mass 0.0 -> 1

Commit message: collision

File: src/agv_ugv/ugv/src/urdf/leo.urdf (robot description, URDF)
Before this commit: robot leo, 12 links, 11 joints
Links:
- link chassis: geometry collision box size=0.25 0.25 0.1; visual mesh filename=package://ugv/src/meshes/Chassis.dae

Commit message: marker

File: src/agv_ugv/ugv/src/urdf/leo.urdf (robot description, URDF)
Before this commit: robot leo, 12 links, 11 joints
Links:
- link aruco: geometry visual mesh filename=package://ugv/src/meshes/Marker1.dae scale=0.6 0.6 0.6

Commit message: aruco scale

File: src/agv_ugv/ugv/src/urdf/leo.urdf (robot description, URDF)
Before this commit: robot leo, 12 links, 11 joints
Links:
- link aruco: geometry visual mesh filename=package://ugv/src/meshes/Marker4.dae scale=0.6 0.6 0.6
Joints:
- joint aruco_joint: origin xyz=0.0 -0.13  0.03 rpy=0.0 0.0 0.0 -> xyz=0.0 -0.15  0.03 rpy=0.0 0.0 0.0
